File: PCB/PCB.kicad_sch (KiCad schematic)
At the start: 30 parts, among them J1 USB_A, SW1 SW_Push, U1 AP2112K-3.3, U2 RP2040, U3 W25Q128JVS, X1 ABM8-272-T3

Commit message: journal for yesterday and schematic done except for battery and stuff
Parts:
- removed C1, C10, C2, C9: 1uF, symbol Device:C
- removed C11, C12, C15, C3, C4, C5, C6, C7, C8: 0.1uF, symbol Device:C
- removed C13, C14: 15pF, symbol Device:C
- removed C16: 10uF, symbol Device:C
- removed H1, H2: MountingHole, symbol Mechanical:MountingHole
- removed J1: USB_A, Connector_USB:USB_A_CNCTech_1001-011-01101_Horizontal, symbol Connector:USB_A
- removed R1: 10K, symbol Device:R
- removed R2, R3: 27, symbol Device:R
- removed R4, R6: 1k, symbol Device:R
- removed R5: DNP, symbol Device:R
- removed SW1: SW_Push, symbol Switch:SW_Push
- removed U1: AP2112K-3.3, Package_TO_SOT_SMD:SOT-23-5, symbol Regulator_Linear:AP2112K-3.3
- removed U2: RP2040, Package_DFN_QFN:QFN-56-1EP_7x7mm_P0.4mm_EP3.2x3.2mm, symbol MCU_RaspberryPi:RP2040
- removed U3: W25Q128JVS, Package_SO:SOIC-8_5.3x5.3mm_P1.27mm, symbol Memory_Flash:W25Q128JVS
- removed X1: ABM8-272-T3, ABM8-272-T3_ABR, symbol Crystal:ABM8-272-T3
Other:
- added sheet Dongle (dongle.kicad_sch)
- added sheet Keyboard (keyboard.kicad_sch)
