File: dongle_pcb/_autosave-dongle_pcb.kicad_sch (KiCad schematic)
At the start: 16 parts, among them J2 USB_A_PCB_Edge_receptacle, SW1 TS-1077S-01726, SW2 TS-1077S-01726, U1 ESP-M2, U2 AP2112K-3.3, U3 CH340G, Y1 12MHz

Commit message: stuff
Parts:
- U2: footprint Package_TO_SOT_SMD:SOT-23-5_HandSoldering -> Package_TO_SOT_SMD:SOT-23-5
Changed lines of the file:
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@@
 			)
 		)
-		(property "Footprint" "Package_TO_SOT_SMD:SOT-23-5_HandSoldering"
+		(property "Footprint" "Package_TO_SOT_SMD:SOT-23-5"
 			(at 139.7 137.795 0)
 			(effects
