File: dongle_pcb/dongle_pcb.kicad_pcb (KiCad board)
At the start: 2 copper layers, 14 x 12 mm, 16 parts, among them J2 USB_A_PCB_Edge_receptacle, SW1 TS-1077S-01726, SW2 TS-1077S-01726, U1 ESP-M2, U2 AP2112K-3.3, U3 CH340G, Y1 12MHz

Commit message: stuff
Parts:
- R4: footprint Capacitor_SMD:C_0603_1608Metric_Pad1.08x0.95mm_HandSolder -> Capacitor_SMD:C_0603_1608Metric
- U2: footprint Package_TO_SOT_SMD:SOT-23-5_HandSoldering -> Package_TO_SOT_SMD:SOT-23-5
Routing:
- net GND: track 0.00 -> 49.7 mm, vias 0 -> 8
- net +3.3V: track 0.00 -> 44.4 mm, vias 0 -> 3
- net Net-(U1-RST): track 0.00 -> 28.9 mm, vias 0 -> 3
- net Net-(U3-XO): track 0.00 -> 28.5 mm, vias 0 -> 2
- net Net-(U3-XI): track 0.00 -> 21.0 mm, vias 0 -> 4
- net Net-(U1-GPIO0): track 0.00 -> 20.5 mm, vias 0 -> 3
- net Net-(U1-GPIO2): track 0.00 -> 17.5 mm
- net D+: track 0.00 -> 12.9 mm
- net Net-(U1-TX): track 0.00 -> 9.04 mm, vias 0 -> 1
- net D-: track 0.00 -> 7.73 mm, vias 0 -> 2
- net Net-(U2-EN): track 0.00 -> 7.73 mm, vias 0 -> 2
- net Net-(U1-RX): track 0.00 -> 7.02 mm, vias 0 -> 1
- net VBUS: track 0.00 -> 4.71 mm, vias 0 -> 2
- net unconnected-(SW2-Pad5): track 0.00 -> 3.50 mm
- net unconnected-(SW1-Pad5): track 0.00 -> 3.50 mm
- added copper zone on B.Cu, net GND
- added copper zone on F.Cu, net GND
Other:
- board size 14 x 12 mm -> 20.1 x 12.6 mm
